Commit message: Replace mesh files

File: robots/panda_arm.xacro (robot description, xacro)
@@ -24,14 +24,14 @@
         <origin rpy="0 0 0" xyz="0 0 0"/>
         <geometry>
-          <mesh filename="package://${package_name}/meshes/link0.STL"/>
-        </geometry>
-        <material name="">
-          <color rgba="1 1 1 1"/>
-        </material>
-      </visual>
-      <collision>
-        <origin rpy="0 0 0" xyz="0 0 0"/>
-        <geometry>
-          <mesh filename="package://${package_name}/meshes/link0_collision.STL"/>
+          <mesh filename="package://${package_name}/meshes/visual/link0.dae"/>
+        </geometry>
+        <material name="">
+          <color rgba="1 1 1 1"/>
+        </material>
+      </visual>
+      <collision>
+        <origin rpy="0 0 0" xyz="0 0 0"/>
+        <geometry>
+          <mesh filename="package://${package_name}/meshes/collision/ link0.stl"/>
         </geometry>
       </collision>
@@ -46,14 +46,14 @@
         <origin rpy="0 0 0" xyz="0 0 0"/>
         <geometry>
-          <mesh filename="package://${package_name}/meshes/link1.STL"/>
-        </geometry>
-        <material name="">
-          <color rgba="1 1 1 1"/>
-        </material>
-      </visual>
-      <collision>
-        <origin rpy="0 0 0" xyz="0 0 0"/>
-        <geometry>
-          <mesh filename="package://${package_name}/meshes/link1_collision.STL"/>
+          <mesh filename="package://${package_name}/meshes/visual/link1.dae"/>
+        </geometry>
+        <material name="">
+          <color rgba="1 1 1 1"/>
+        </material>
+      </visual>
+      <collision>
+        <origin rpy="0 0 0" xyz="0 0 0"/>
+        <geometry>
+          <mesh filename="package://${package_name}/meshes/collision/link1.stl"/>
         </geometry>
       </collision>
@@ -76,14 +76,14 @@
         <origin rpy="0 0 0" xyz="0 0 0"/>
         <geometry>
-          <mesh filename="package://${package_name}/meshes/link2.STL"/>
-        </geometry>
-        <material name="">
-          <color rgba="1 1 1 1"/>
-        </material>
-      </visual>
-      <collision>
-        <origin rpy="0 0 0" xyz="0 0 0"/>
-        <geometry>
-          <mesh filename="package://${package_name}/meshes/link2_collision.STL"/>
+          <mesh filename="package://${package_name}/meshes/visual/link2.dae"/>
+        </geometry>
+        <material name="">
+          <color rgba="1 1 1 1"/>
+        </material>
+      </visual>
+      <collision>
+        <origin rpy="0 0 0" xyz="0 0 0"/>
+        <geometry>
+          <mesh filename="package://${package_name}/meshes/collision/link2.stl"/>
         </geometry>
       </collision>
@@ -106,14 +106,14 @@
         <origin rpy="0 0 0" xyz="0 0 0"/>
         <geometry>
-          <mesh filename="package://${package_name}/meshes/link3.STL"/>
-        </geometry>
-        <material name="">
-          <color rgba="1 1 1 1"/>
-        </material>
-      </visual>
-      <collision>
-        <origin rpy="0 0 0" xyz="0 0 0"/>
-        <geometry>
-          <mesh filename="package://${package_name}/meshes/link3_collision.STL"/>
+          <mesh filename="package://${package_name}/meshes/visual/link3.dae"/>
+        </geometry>
+        <material name="">
+          <color rgba="1 1 1 1"/>
+        </material>
+      </visual>
+      <collision>
+        <origin rpy="0 0 0" xyz="0 0 0"/>
+        <geometry>
+          <mesh filename="package://${package_name}/meshes/collision/link3.stl"/>
         </geometry>
       </collision>
@@ -136,14 +136,14 @@
         <origin rpy="0 0 0" xyz="0 0 0"/>
         <geometry>
-          <mesh filename="package://${package_name}/meshes/link4.STL"/>
-        </geometry>
-        <material name="">
-          <color rgba="1 1 1 1"/>
-        </material>
-      </visual>
-      <collision>
-        <origin rpy="0 0 0" xyz="0 0 0"/>
-        <geometry>
-          <mesh filename="package://${package_name}/meshes/link4_collision.STL"/>
+          <mesh filename="package://${package_name}/meshes/visual/link4.dae"/>
+        </geometry>
+        <material name="">
+          <color rgba="1 1 1 1"/>
+        </material>
+      </visual>
+      <collision>
+        <origin rpy="0 0 0" xyz="0 0 0"/>
+        <geometry>
+          <mesh filename="package://${package_name}/meshes/collision/link4.stl"/>
         </geometry>
       </collision>
@@ -166,14 +166,14 @@
         <origin rpy="0 0 0" xyz="0 0 0"/>
         <geometry>
-          <mesh filename="package://${package_name}/meshes/link5.STL"/>
-        </geometry>
-        <material name="">
-          <color rgba="1 1 1 1"/>
-        </material>
-      </visual>
-      <collision>
-        <origin rpy="0 0 0" xyz="0 0 0"/>
-        <geometry>
-          <mesh filename="package://${package_name}/meshes/link5_collision.STL"/>
+          <mesh filename="package://${package_name}/meshes/visual/link5.dae"/>
+        </geometry>
+        <material name="">
+          <color rgba="1 1 1 1"/>
+        </material>
+      </visual>
+      <collision>
+        <origin rpy="0 0 0" xyz="0 0 0"/>
+        <geometry>
+          <mesh filename="package://${package_name}/meshes/collision/link5.stl"/>
         </geometry>
       </collision>
@@ -196,14 +196,14 @@
         <origin rpy="0 0 0" xyz="0 0 0"/>
         <geometry>
-          <mesh filename="package://${package_name}/meshes/link6.STL"/>
-        </geometry>
-        <material name="">
-          <color rgba="1 1 1 1"/>
-        </material>
-      </visual>
-      <collision>
-        <origin rpy="0 0 0" xyz="0 0 0"/>
-        <geometry>
-          <mesh filename="package://${package_name}/meshes/link6_collision.STL"/>
+          <mesh filename="package://${package_name}/meshes/visual/link6.dae"/>
+        </geometry>
+        <material name="">
+          <color rgba="1 1 1 1"/>
+        </material>
+      </visual>
+      <collision>
+        <origin rpy="0 0 0" xyz="0 0 0"/>
+        <geometry>
+          <mesh filename="package://${package_name}/meshes/collision/link6.stl"/>
         </geometry>
       </collision>
@@ -226,14 +226,14 @@
         <origin rpy="0 0 0" xyz="0 0 0"/>
         <geometry>
-          <mesh filename="package://${package_name}/meshes/link7.STL"/>
-        </geometry>
-        <material name="">
-          <color rgba="1 1 1 1"/>
-        </material>
-      </visual>
-      <collision>
-        <origin rpy="0 0 0" xyz="0 0 0"/>
-        <geometry>
-          <mesh filename="package://${package_name}/meshes/link7_collision.STL"/>
+          <mesh filename="package://${package_name}/meshes/visual/link7.dae"/>
+        </geometry>
+        <material name="">
+          <color rgba="1 1 1 1"/>
+        </material>
+      </visual>
+      <collision>
+        <origin rpy="0 0 0" xyz="0 0 0"/>
+        <geometry>
+          <mesh filename="package://${package_name}/meshes/collision/link7.stl"/>
         </geometry>
       </collision>
@@ -241,5 +241,5 @@
     <joint name="${arm_id}_joint7" type="revolute">
       <safety_controller k_position="100.0" k_velocity="40.0" soft_lower_limit="-2.818745" soft_upper_limit="2.818745"/>
-      <origin rpy="${pi/2} ${-pi/4} 0" xyz="0.088 0 0"/>
+      <origin rpy="${pi/2} 0 0" xyz="0.088 0 0"/> <!-- y za orijentaciju ruke na -pi/4 -->
       <parent link="${arm_id}_link6"/>
       <child link="${arm_id}_link7"/>

Commit message: Fix broken joints.

File: robots/panda_arm.xacro (robot description, xacro)
@@ -150,10 +150,12 @@
     </link>
     <joint name="${arm_id}_joint4" type="revolute">
-      <safety_controller k_position="100.0" k_velocity="40.0" soft_lower_limit="-3.0718" soft_upper_limit="-0.0698"/>
+      <safety_controller k_position="100.0" k_velocity="40.0" soft_lower_limit="-3.0718" soft_upper_limit="0.0698"/>
+      <!-- soft_upper_limitr should be -0.0698, but that brakes simulation when initial position for this joint is 0.0 -->
       <origin rpy="${pi/2} 0 0" xyz="0.0825 0 0"/>
       <parent link="${arm_id}_link3"/>
       <child link="${arm_id}_link4"/>
       <axis xyz="0 0 1"/>
-      <limit effort="87" lower="-3.0718" upper="-0.0698" velocity="2.1750"/>
+      <limit effort="87" lower="-3.0718" upper="0.0698" velocity="2.1750"/>
+      <!-- upper should be -0.0698, but that brakes simulation when initial position for this joint is 0.0 -->
     </joint>
     <link name="${arm_id}_link5">
