Commit message: Add more realistic inertial parameters and semi-optimize PID gains.

File: robots/hand.gazebo.xacro (robot description, xacro)
@@ -7,5 +7,5 @@
     <type>transmission_interface/SimpleTransmission</type>
     <joint name="${ns}_finger_joint1">
-      <hardwareInterface>hardware_interface/EffortJointInterface</hardwareInterface>
+      <hardwareInterface>hardware_interface/PositionJointInterface</hardwareInterface>
     </joint>
     <actuator name="${ns}_finger_joint1_motor">
@@ -16,5 +16,5 @@
     <type>transmission_interface/SimpleTransmission</type>
     <joint name="${ns}_finger_joint2">
-      <hardwareInterface>hardware_interface/EffortJointInterface</hardwareInterface>
+      <hardwareInterface>hardware_interface/PositionJointInterface</hardwareInterface>
     </joint>
     <actuator name="${ns}_finger_joint2_motor">

File: robots/hand.xacro (robot description, xacro)
@@ -16,7 +16,7 @@
     <link name="${ns}_hand">
       <inertial>
-        <mass value="0.3" />
+        <mass value="0.73" />
         <origin xyz="0 0.0015244 0.0275912" rpy="0 0 0" />
-        <inertia ixx="0.0011447680686" ixy="0.0" ixz="0.0" iyy="0.000164397289864" iyz="0.0" izz="0.00105360839109" />
+        <inertia ixx="0.00278560230025" ixy="0.0" ixz="0.0" iyy="0.000400033405336" iyz="0.0" izz="0.00256378041832" />
       </inertial>
       <visual>

File: robots/panda_arm.xacro (robot description, xacro)
@@ -17,7 +17,7 @@
     <link name="${arm_id}_link0">
       <inertial>
-        <mass value="1.2" />
+        <mass value="2.92" />
         <origin xyz="-0.025566 -2.88e-05 0.057332" rpy="0 0 0" />
-        <inertia ixx="0.00321464142876" ixy="-6.41883382175e-06" ixz="-0.000517831800505" iyy="0.00448060158136" iyz="4.44796677541e-06" izz="0.00420639057326" />
+        <inertia ixx="0.00782229414331" ixy="-1.56191622996e-05" ixz="-0.00126005738123" iyy="0.0109027971813" iyz="1.08233858202e-05" izz="0.0102355503949" />
       </inertial>
       <visual>
@@ -39,7 +39,7 @@
     <link name="${arm_id}_link1">
       <inertial>
-        <mass value="2.0" />
+        <mass value="2.74" />
         <origin xyz="0 -0.0324958 -0.0675818" rpy="0 0 0" />
-        <inertia ixx="0.0131691210426" ixy="0.0" ixz="0.0" iyy="0.0116157716709" iyz="0.00341302369431" izz="0.00453058997903" />
+        <inertia ixx="0.0180416958283" ixy="0.0" ixz="0.0" iyy="0.0159136071891" iyz="0.0046758424612" izz="0.00620690827127" />
       </inertial>
       <visual>
@@ -69,7 +69,7 @@
     <link name="${arm_id}_link2">
       <inertial>
-        <mass value="2.0" />
+        <mass value="2.74" />
         <origin xyz="0 -0.06861 0.0322285" rpy="0 0 0" />
-        <inertia ixx="0.0133471665898" ixy="0.0" ixz="0.0" iyy="0.00453546292829" iyz="-0.00345141767814" izz="0.0117893683438" />
+        <inertia ixx="0.0182856182281" ixy="0.0" ixz="0.0" iyy="0.00621358421175" iyz="-0.00472844221905" izz="0.0161514346309" />
       </inertial>
       <visual>
@@ -99,7 +99,7 @@
     <link name="${arm_id}_link3">
       <inertial>
-        <mass value="2.0" />
+        <mass value="2.38" />
         <origin xyz="0.0469893 0.0316374 -0.031704" rpy="0 0 0" />
-        <inertia ixx="0.00648215656226" ixy="-0.00208815651376" ixz="-0.00279115614313" iyy="0.00831183200611" iyz="-0.00183021976037" izz="0.00682120637365" />
+        <inertia ixx="0.00771376630908" ixy="-0.00248490625138" ixz="-0.00332147581033" iyy="0.00989108008727" iyz="-0.00217796151484" izz="0.00811723558464" />
       </inertial>
       <visual>
@@ -129,7 +129,7 @@
     <link name="${arm_id}_link4">
       <inertial>
-        <mass value="2.0" />
+        <mass value="2.38" />
         <origin xyz="-0.0360446 0.0336853 0.031882" rpy="0 0 0" />
-        <inertia ixx="0.00671986454733" ixy="0.00291676949762" ixz="-0.00202708355458" iyy="0.00693605634688" iyz="0.00198129448841" izz="0.00861470624749" />
+        <inertia ixx="0.00799663881132" ixy="0.00347095570217" ixz="-0.00241222942995" iyy="0.00825390705278" iyz="0.00235774044121" izz="0.0102515004345" />
       </inertial>
       <visual>
@@ -161,7 +161,7 @@
     <link name="${arm_id}_link5">
       <inertial>
-        <mass value="2.0" />
+        <mass value="2.74" />
         <origin xyz="0 0.0610427 -0.104176" rpy="0 0 0" />
-        <inertia ixx="0.0221688865058" ixy="4.74659552633e-07" ixz="-7.67366276757e-06" iyy="0.0210768530951" iyz="-0.00566170398384" izz="0.00324185442455" />
+        <inertia ixx="0.030371374513" ixy="6.50283587108e-07" ixz="-1.05129179916e-05" iyy="0.0288752887402" iyz="-0.00775653445787" izz="0.00444134056164" />
       </inertial>
       <visual>
@@ -191,7 +191,7 @@
     <link name="${arm_id}_link6">
       <inertial>
-        <mass value="1.0" />
+        <mass value="1.55" />
         <origin xyz="0.0510509 0.009108 0.0106343" rpy="0 0 0" />
-        <inertia ixx="0.00195700935727" ixy="-0.000282114106779" ixz="0.000405972448308" iyy="0.00260954781656" iyz="8.41754974355e-05" izz="0.00360151152283" />
+        <inertia ixx="0.00303336450376" ixy="-0.000437276865508" ixz="0.000629257294877" iyy="0.00404479911567" iyz="0.000130472021025" izz="0.00558234286039" />
       </inertial>
       <visual>
@@ -221,7 +221,7 @@
     <link name="${arm_id}_link7">
       <inertial>
-        <mass value="0.2" />
+        <mass value="0.54" />
         <origin xyz="0.0109695 0.0107965 0.0650411" rpy="0 0 0" />
-        <inertia ixx="0.000329210698897" ixy="-4.53299061184e-05" ixz="1.4766660358e-05" iyy="0.000328889397494" iyz="-3.4586115378e-05" izz="0.000265808689222" />
+        <inertia ixx="0.000888868887021" ixy="-0.00012239074652" ixz="3.98699829666e-05" iyy="0.000888001373233" iyz="-9.33825115206e-05" izz="0.0007176834609" />
       </inertial>
       <visual>
